Commit message: lidar rviz visualization fix

File: src/description/urdf/common_properties.xacro (robot description, xacro)
@@ -3,4 +3,7 @@
     <material name="blue">
         <color rgba="0 0 0.5 1" />
+    </material>
+    <material name="red">
+        <color rgba="1 0 00 1" />
     </material>
     <material name="grey">

File: src/description/urdf/lidar.xacro (robot description, xacro)
@@ -8,5 +8,5 @@
         <cylinder radius="${lidar_radius}" length="${lidar_length}" />
       </geometry>
-      <material name="grey" />
+      <material name="red" />
     </visual>
     <collision>
@@ -23,5 +23,5 @@
   </joint>
   <gazebo reference="lidar_link">
-    <material>Gazebo/Purple</material>
+    <material>Gazebo/Red</material>
     <sensor name="lidar" type="ray">
       <pose>0 0 0 0 0 0</pose>
@@ -46,5 +46,5 @@
       </ros>
       <output_type>sensor_msgs/LaserScan</output_type>
-      <frame_name>lidar_frame</frame_name>
+      <frame_name>lidar_link</frame_name>
       </plugin>
     </sensor>
